File: hardware/ft2232_interface.kicad_sch (KiCad schematic)
At the start: 64 parts, among them J27 Conn_02x20_Odd_Even, U10 93LC56BT-E/OT, U7 FT2232HQ, Y1 12MHz crystal +/- 30ppm max 1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

Commit message: Routing and several design fixes
Signed-off-by: Miguel Angel Ajo Pelayo <majopela@redhat.com>
Signed-off-by: Ricardo Noriega <rnoriega@redhat.com>
Parts:
- added R?: NC 10k, Resistor_SMD:R_0402_1005Metric, symbol Device:R
- R?: value 12k -> 12k 1%
Connections:
- net +3.3V: now also R?.2
- net BC7: now also R?.1
- net FT2232_DN: now also U7.7 (DM); no longer U7.8 (DP)
- net FT2232_DP: now also U7.8 (DP); no longer U7.7 (DM)
- net _nPWREN renamed _PWREN
- net nPWREN renamed PWREN
Other:
- note added: "*PWRSAV#=1 NORMAL OPERATION"
Changed lines of the file:
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@@
   (junction (at 139.065 36.83) (diameter 0) (color 0 0 0 0)
   )
+  (junction (at 191.77 144.145) (diameter 0) (color 0 0 0 0)
+  )
   (junction (at 126.365 161.925) (diameter 0) (color 0 0 0 0)
   )
@@
     (stroke (width 0) (type default))
   )
+  (wire (pts (xy 191.77 146.05) (xy 217.17 146.05))
+    (stroke (width 0) (type default))
+  )
+  (wire (pts (xy 191.77 144.145) (xy 196.215 144.145))
+    (stroke (width 0) (type default))
+  )
   (wire (pts (xy 187.325 151.765) (xy 196.85 151.765))
     (stroke (width 0) (type default))
@@
     (stroke (width 0) (type default))
   )
-  (wire (pts (xy 187.325 144.145) (xy 196.215 144.145))
+  (wire (pts (xy 187.325 144.145) (xy 191.77 144.145))
     (stroke (width 0) (type default))
   )
@@
     (stroke (width 0) (type default))
   )
+  (wire (pts (xy 224.79 146.05) (xy 227.584 146.05))
+    (stroke (width 0) (type default))
+  )
   (wire (pts (xy 55.88 67.945) (xy 55.88 69.85))
     (stroke (width 0) (type default))
@@
     (stroke (width 0) (type default))
   )
+  (wire (pts (xy 191.77 144.145) (xy 191.77 146.05))
+    (stroke (width 0) (type default))
+  )
   (wire (pts (xy 229.235 128.905) (xy 238.125 128.905))
     (stroke (width 0) (type default))
@@
     (stroke (width 0) (type default))
   )
+  (text "*PWRSAV#=1 NORMAL OPERATION\n" (at 223.647 149.86 0)
+    (effects (font (size 1.27 1.27)) (justify left bottom))
+  )
   (label "AD0" (at 189.865 57.785 0) (fields_autoplaced)
     (effects (font (size 1.27 1.27)) (justify left bottom))
@@
     (effects (font (size 1.27 1.27)) (justify left bottom))
   )
-  (label "_nPWREN" (at 210.185 149.225 0) (fields_autoplaced)
+  (label "_PWREN" (at 210.185 149.225 0) (fields_autoplaced)
     (effects (font (size 1.27 1.27)) (justify left bottom))
   )
@@
     (effects (font (size 1.27 1.27)) (justify left bottom))
   )
-  (label "nPWREN" (at 187.96 149.225 0) (fields_autoplaced)
+  (label "PWREN" (at 187.96 149.225 0) (fields_autoplaced)
     (effects (font (size 1.27 1.27)) (justify left bottom))
   )
@@
     (effects (font (size 1.27 1.27)) (justify left bottom))
   )
-  (label "_nPWREN" (at 229.235 128.905 0) (fields_autoplaced)
-    (effects (font (size 1.27 1.27)) (justify left bottom))
-  )
   (label "_AD6" (at 232.41 88.265 0) (fields_autoplaced)
     (effects (font (size 1.27 1.27)) (justify left bottom))
@@
     (effects (font (size 1.27 1.27)) (justify left bottom))
   )
+  (label "_PWREN" (at 230.759 128.905 0) (fields_autoplaced)
+    (effects (font (size 1.27 1.27)) (justify left bottom))
+  )
   (label "_BC4" (at 231.775 121.285 0) (fields_autoplaced)
     (effects (font (size 1.27 1.27)) (justify left bottom))
@@
     (effects (font (size 1.27 1.27)) (justify left bottom))
   )
-  (hierarchical_label "FT2232_DP" (shape bidirectional) (at 33.02 83.185 180) (fields_autoplaced)
-    (effects (font (size 1.27 1.27)) (justify right))
-  )
   (hierarchical_label "FT2232_EECS" (shape input) (at 34.29 126.365 180) (fields_autoplaced)
     (effects (font (size 1.27 1.27)) (justify right))
@@
     (effects (font (size 1.27 1.27)) (justify right))
   )
-  (hierarchical_label "FT2232_DN" (shape bidirectional) (at 33.02 85.725 180) (fields_autoplaced)
-    (effects (font (size 1.27 1.27)) (justify right))
-  )
   (hierarchical_label "FT2232_EECLK" (shape input) (at 119.38 122.555 180) (fields_autoplaced)
     (effects (font (size 1.27 1.27)) (justify right))
@@
     (effects (font (size 1.27 1.27)) (justify right))
   )
+  (hierarchical_label "FT2232_DN" (shape bidirectional) (at 33.02 83.185 180) (fields_autoplaced)
+    (effects (font (size 1.27 1.27)) (justify right))
+  )
+  (hierarchical_label "FT2232_DP" (shape bidirectional) (at 33.02 85.725 180) (fields_autoplaced)
+    (effects (font (size 1.27 1.27)) (justify right))
+  )
   (symbol (lib_id "power:+3.3V") (at 88.9 113.03 0) (unit 1)
     (in_bom yes) (on_board yes) (dnp no)
@@
       (effects (font (size 1.27 1.27)))
     )
-    (property "Value" "12k" (at 119.38 95.885 90)
+    (property "Value" "12k 1%" (at 119.38 95.885 90)
       (effects (font (size 1.27 1.27)))
     )
@@
     )
   )
+  (symbol (lib_id "Device:R") (at 220.98 146.05 90) (unit 1)
+    (in_bom yes) (on_board yes) (dnp no)
+    (property "Reference" "R?" (at 226.695 144.78 90)
+      (effects (font (size 1.27 1.27)))
+    )
+    (property "Value" "NC 10k" (at 220.98 146.05 90)
+      (effects (font (size 1.27 1.27)))
+    )
+    (property "Footprint" "Resistor_SMD:R_0402_1005Metric" (at 220.98 147.828 90)
+      (effects (font (size 1.27 1.27)) hide)
+    )
+    (property "Datasheet" "~" (at 220.98 146.05 0)
+      (effects (font (size 1.27 1.27)) hide)
+    )
+    (pin "1")
+    (pin "2")
+    (instances
+      (project "jumpstarter"
+        (path "/5e49fb74-0a9b-4946-8b59-2b8244d10fd9"
+          (reference "R?") (unit 1)
+        )
+        (path "/5e49fb74-0a9b-4946-8b59-2b8244d10fd9/0a246f5a-dd08-4f47-947a-3b89ae06d789"
+          (reference "R?") (unit 1)
+        )
+        (path "/5e49fb74-0a9b-4946-8b59-2b8244d10fd9/07a45a66-b9c7-469a-85fe-580b6ce09702"
+          (reference "R118") (unit 1)
+        )
+      )
+    )
+  )
   (symbol (lib_id "Device:R") (at 200.025 121.285 90) (unit 1)
     (in_bom yes) (on_board yes) (dnp no)
@@
         )
       )
+    )
+  )
+  (symbol (lib_id "power:+3.3V") (at 227.584 146.05 270) (unit 1)
+    (in_bom yes) (on_board yes) (dnp no)
+    (property "Reference" "#PWR013" (at 223.774 146.05 0)
+      (effects (font (size 1.27 1.27)) hide)
+    )
+    (property "Value" "+3.3V" (at 232.664 146.05 0)
+      (effects (font (size 1.27 1.27)))
+    )
+    (property "Footprint" "" (at 227.584 146.05 0)
+      (effects (font (size 1.27 1.27)) hide)
+    )
+    (property "Datasheet" "" (at 227.584 146.05 0)
+      (effects (font (size 1.27 1.27)) hide)
+    )
+    (pin "1")
+    (instances
+      (project "jumpstarter"
+        (path "/5e49fb74-0a9b-4946-8b59-2b8244d10fd9"
+          (reference "#PWR013") (unit 1)
+        )
+        (path "/5e49fb74-0a9b-4946-8b59-2b8244d10fd9/c1addf8b-26b2-43fb-875c-11d76afd1403"
+          (reference "#PWR0109") (unit 1)
+        )
+        (path "/5e49fb74-0a9b-4946-8b59-2b8244d10fd9/07a45a66-b9c7-469a-85fe-580b6ce09702"
+          (reference "#PWR0223") (unit 1)
+        )
+      )

Commit message: Almost ready 2.0.0
Parts:
- C23: MFN (none) -> CL10B104KB8NNNC
- C66, C67: MFN (none) -> UMK105CG270JVHF; MPN (none) -> UMK105CG270JVHF
- C? (x2): footprint Capacitor_SMD:C_0603_1608Metric_Pad1.08x0.95mm_HandSolder -> Capacitor_SMD:C_0603_1608Metric; MFN (none) -> CSA0603X5R475K6R3JT; MPN (none) -> CSA0603X5R475K6R3JT
- C?: footprint Capacitor_SMD:C_0603_1608Metric_Pad1.08x0.95mm_HandSolder -> Capacitor_SMD:C_0603_1608Metric; MFN (none) -> CL10A335KP8NNNC; MPN (none) -> CL10A335KP8NNNC
- J27: MFN (none) -> 95157-440LF
- L2: MFN (none) -> BLM15AG121SH1D
- R11, R? (x30): MFN (none) -> RTT021000FTH; MPN (none) -> RTT021000FTH
- R11, R?: MFN (none) -> NC; MPN (none) -> NC
- R? (x2): MFN (none) -> RTT02202JTH; MPN (none) -> RTT02202JTH
- R?: MFN (none) -> RTT021202FTH; MPN (none) -> RTT021202FTH
- R? (x3): MFN (none) -> RTT02103JTH; MPN (none) -> RTT02103JTH
- U10: Link (none) -> https://www2.mouser.com/ProductDetail/Microchip-Technology/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; MFN (none) -> 93LC56BT-E/OT
- U7: MFN (none) -> FT2232HQ-REEL
- Y1: value 12MHz crystal +/- 30ppm max 12pf -> Cristales 12.000 MHZ 10PF; MFN (none) -> ABM8G-12.000MHZ-4Y-T3; MPN X1E000021013900 -> ABM8G-12.000MHZ-4Y-T3
