File: hardware/jumpstarter.kicad_sch (KiCad schematic)
At the start: 66 parts, among them J10 Conn_01x02_Pin, J11 Conn_01x02_Pin, J12 Conn_01x02_Pin, J13 Conn_01x02_Pin, J14 Conn_01x02_Pin, J15 Conn_01x02_Pin, J6 Conn_01x05_Pin, P1 USB_C_Plug_USB2.0, SW1 SW_Push, SW2 SW_Push, SW3 SW_Push, U1 STM32F411CEUx, U2 AP2127N-3.3, U3 AP2127N-3.3, Y2 25 Mhz Crystal

Commit message: WIP 1.1
Parts:
- removed 5V1: TestPoint, TestPoint:TestPoint_Pad_D1.0mm, symbol Connector:TestPoint
- removed C8, C9: 12pF, Capacitor_SMD:C_0603_1608Metric_Pad1.08x0.95mm_HandSolder, symbol Device:C
- removed P1: USB_C_Plug_USB2.0, Connector_USB:USB_C_Receptacle_G-Switch_GT-USB-7010ASV, symbol Connector:USB_C_Plug_USB2.0
- removed R17, R18: 10, Resistor_SMD:R_0603_1608Metric, symbol Device:R
- removed R19: 5k1, Resistor_SMD:R_0603_1608Metric, symbol Device:R
- removed Y2: 25 Mhz Crystal, Oscillator:Oscillator_SMD_EuroQuartz_XO32-4Pin_3.2x2.5mm, symbol Device:Crystal_GND24
Connections:
- net XTALI: no longer names the net of U1.6 (PH1)
- net XTALO renamed CLK_25MHz
Other:
- added sheet USB 3.2 Gen2 front-hub (usb3_hub.kicad_sch)

Commit message: Started routing USB3 diff pairs
Parts:
- removed 3v3, 3v3A1, TP3, TP4, TP7, TP9: TestPoint, TestPoint:TestPoint_Pad_D1.0mm, symbol Connector:TestPoint
- removed C1, C2, C3, C4: 1uF, Capacitor_SMD:C_0603_1608Metric_Pad1.08x0.95mm_HandSolder, symbol Device:C
- removed H17, H18: cable strap hole, MountingHole:MountingHole_4.3mm_M4_Pad_Via, symbol Mechanical:MountingHole
- removed J10, J11, J12, J13, J14, J15: Conn_01x02_Pin, Connector_PinHeader_2.54mm:PinHeader_1x02_P2.54mm_Vertical, symbol Connector:Conn_01x02_Pin
- removed J6: Conn_01x05_Pin, Connector_PinHeader_2.54mm:PinHeader_1x05_P2.54mm_Vertical, symbol Connector:Conn_01x05_Pin
- removed L1, L3: 10uH, Inductor_SMD:L_0805_2012Metric, symbol Device:L_Ferrite
- removed U2, U3: AP2127N-3.3, Package_TO_SOT_SMD:SOT-23, symbol Regulator_Linear:AP2127N-3.3
- added C66, C67: 12pF, Capacitor_SMD:C_0402_1005Metric, symbol Device:C
- added C73, C75: 1uF, Capacitor_SMD:C_0603_1608Metric_Pad1.08x0.95mm_HandSolder, symbol Device:C
- added C74, C76: 100nF, Capacitor_SMD:C_0402_1005Metric, symbol Device:C
- added FID1, FID2, FID3, FID4, FID5, FID6: Fiducial, Fiducial:Fiducial_0.5mm_Mask1mm, symbol Mechanical:Fiducial
- added J20: SPI/TPM connector, Connector_PinHeader_2.54mm:PinHeader_2x05_P2.54mm_Vertical, symbol Connector_Generic:Conn_02x05_Odd_Even
- added J21: I2C connector, Connector_PinHeader_2.54mm:PinHeader_2x03_P2.54mm_Vertical, symbol Connector_Generic:Conn_02x03_Odd_Even
- added J22: NC, Connector:Tag-Connect_TC2050-IDC-FP_2x05_P1.27mm_Vertical, symbol Connector_Generic:Conn_02x05_Odd_Even
- added J28: CASE CONNECTORS, Connector_PinHeader_2.54mm:PinHeader_2x06_P2.54mm_Vertical, symbol Connector_Generic:Conn_02x06_Odd_Even
- added R109, R110, R111, R112: 470, Resistor_SMD:R_0402_1005Metric, symbol Device:R
- added Y1: 25 Mhz Crystal +/- 10ppm, Oscillator:Oscillator_SMD_EuroQuartz_XO32-4Pin_3.2x2.5mm, symbol Device:Crystal_GND24
- C14, C15, C17, C18: footprint Capacitor_SMD:C_0603_1608Metric_Pad1.08x0.95mm_HandSolder -> Capacitor_SMD:C_0402_1005Metric; MPN (none) -> CL05B104K05NNNC; MPN2 (none) -> TCC0402X7R104M160AT
- C16, C7: footprint Capacitor_SMD:C_0603_1608Metric -> Capacitor_SMD:C_0402_1005Metric; MPN (none) -> CL05B104K05NNNC; MPN2 (none) -> TCC0402X7R104M160AT
- R1, R10, R15, R2, R22: footprint Resistor_SMD:R_0603_1608Metric -> Resistor_SMD:R_0402_1005Metric
- R16, R20, R21, R23: value 1k -> 470; footprint Resistor_SMD:R_0603_1608Metric -> Resistor_SMD:R_0402_1005Metric
- SW2: footprint Button_Switch_SMD:SW_SPST_B3S-1000 -> Button_Switch_THT:SW_Tactile_SPST_Angled_PTS645Vx58-2LFS
Connections:
- net +3.3V: now also C73.2, C74.1, C75.2, C76.1, J20.1 (Pin_1), J21.1 (Pin_1), J21.5 (Pin_5), J22.1 (Pin_1), J28.2 (Pin_2), J28.4 (Pin_4), J28.6 (Pin_6), J28.8 (Pin_8)
- net BUTTON: now also J28.10 (Pin_10)
- net GND: now also C66.1, C67.1, C73.1, C74.2, C75.1, C76.2, J20.4 (Pin_4), J20.9 (Pin_9), J21.3 (Pin_3), J22.10 (Pin_10), J22.2 (Pin_2), J22.4 (Pin_4), J22.6 (Pin_6), J22.7 (Pin_7), J22.8 (Pin_8), J28.11 (Pin_11), J28.9 (Pin_9), R109.1, Y1.2, Y1.4
- net LED0: now also R112.1
- net LED1: now also R111.1
- net LED2: now also R110.1
- net NRST: now also J22.9 (Pin_9), J28.12 (Pin_12)
- net SWCLK: now also J22.5 (Pin_5)
- net SWDIO: now also J22.3 (Pin_3)
- net FT2232_EECLK: now reaches U1.13 (PA3)
- net nRESET_OUT: now reaches U1.18 (PB0)
- net nRESET_OUT: now also J20.2 (Pin_2)
- net FT2232_EECS: now reaches U1.19 (PB1)
- net IRQ_IN: now reaches U1.21 (PB10)
- net IRQ_IN: now also J20.6 (Pin_6), J21.6 (Pin_6)
- net SPI2_NSS: now reaches U1.25 (PB12)
- net SPI2_NSS: now also J20.10 (Pin_10)
- net SPI2_SCK: now reaches U1.26 (PB13)
- net SPI2_SCK: now also J20.7 (Pin_7)
- net SPI2_MISO: now reaches U1.27 (PB14)
- net SPI2_MISO: now also J20.5 (Pin_5)
- net SPI2_MOSI: now reaches U1.28 (PB15)
- net SPI2_MOSI: now also J20.3 (Pin_3)
- net FT2232_EEDATA: now reaches U1.31 (PA10)
- net I2C1_SCL: now reaches U1.45 (PB8)
- net I2C1_SCL: now also J21.2 (Pin_2)
- net I2C1_SDA: now reaches U1.46 (PB9)
- net I2C1_SDA: now also J21.4 (Pin_4)
- net XTALO: now reaches U1.6 (PH1)
- net XTALO: now also C67.2, Y1.3
- net CLK_25MHz renamed XTALI
- net XTALI: now also C66.2, Y1.1
- new net: J28.7 (Pin_7), R112.2
- new net: J28.3 (Pin_3), R110.2
- new net: J28.1 (Pin_1), R109.2
- new net: J28.5 (Pin_5), R111.2
- no-connect marks 0 -> 1
Other:
- added sheet FT2232 (ft2232_interface.kicad_sch)
- added sheet Power (power_supplies.kicad_sch)
- sheet USB 3.2 Gen2 front-hub ports: added DN, DP, PRTCTL, SSRXN, SSRXP, SSTXN, SSTXP, VBUS_UPSTREAM; removed P5_DN, P5_DP, P5_SSRXN, P5_SSRXP, P5_SSTXN, P5_SSTXP
- sheet USB_STORAGE_MUX ports: added HUB_PRTCTL, SHOST_DN, SHOST_DP, SHOST_SSRXN, SHOST_SSRXP, SHOST_SSTXN, SHOST_SSTXP; removed none
- sheet board_control ports: added V_IN_ATX12, V_IN_ATX5; removed none
- note added: "LEDS"
- note added: "RESET"
- moved on the sheet: C10, C14, C15, C16, C17, C18, C7, D1, D2, D3, D4, GND1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

Commit message: Routing and several design fixes
Signed-off-by: Miguel Angel Ajo Pelayo <majopela@redhat.com>
Signed-off-by: Ricardo Noriega <rnoriega@redhat.com>
Connections:
- net GND: no longer C14.2
- net GNDA: now also C14.2
Changed lines of the file:
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@@
+    )
+  )
+  (symbol (lib_id "power:GNDA") (at 271.78 121.92 90) (unit 1)
+    (in_bom yes) (on_board yes) (dnp no) (fields_autoplaced)
+    (property "Reference" "#PWR050" (at 278.13 121.92 0)
+      (effects (font (size 1.27 1.27)) hide)
+    )
+    (property "Value" "GNDA" (at 275.59 121.92 90)
+      (effects (font (size 1.27 1.27)) (justify right))
+    )
+    (property "Footprint" "" (at 271.78 121.92 0)
+      (effects (font (size 1.27 1.27)) hide)
+    )
+    (property "Datasheet" "" (at 271.78 121.92 0)
+      (effects (font (size 1.27 1.27)) hide)
+    )
+    (pin "1")
+    (instances
+      (project "jumpstarter"
+        (path "/5e49fb74-0a9b-4946-8b59-2b8244d10fd9"
+          (reference "#PWR050") (unit 1)
+        )
+      )
     )
   )
@@
     )
   )
-  (symbol (lib_id "power:GND") (at 271.78 121.92 90) (unit 1)
-    (in_bom yes) (on_board yes) (dnp no)
-    (property "Reference" "#PWR047" (at 278.13 121.92 0)
-      (effects (font (size 1.27 1.27)) hide)
-    )
-    (property "Value" "GND" (at 270.51 124.46 90)
-      (effects (font (size 1.27 1.27)) (justify right))
-    )
-    (property "Footprint" "" (at 271.78 121.92 0)
-      (effects (font (size 1.27 1.27)) hide)
-    )
-    (property "Datasheet" "" (at 271.78 121.92 0)
-      (effects (font (size 1.27 1.27)) hide)
-    )
-    (pin "1")
-    (instances
-      (project "jumpstarter"
-        (path "/5e49fb74-0a9b-4946-8b59-2b8244d10fd9"
-          (reference "#PWR047") (unit 1)
-        )
-      )
-    )
-  )
   (symbol (lib_id "Diode:1N4148WT") (at 98.425 40.005 270) (unit 1)
     (in_bom yes) (on_board yes) (dnp no)
@@
       (effects (font (size 1.27 1.27)) (justify left))
     )
-    (pin "SHOST_SSRXP" bidirectional (at 81.28 154.305 180)
-      (effects (font (size 1.27 1.27)) (justify left))
-    )
     (pin "SHOST_SSTXN" bidirectional (at 81.28 148.59 180)
       (effects (font (size 1.27 1.27)) (justify left))
@@
       (effects (font (size 1.27 1.27)) (justify left))
     )
-    (pin "SHOST_SSRXN" bidirectional (at 81.28 151.765 180)
-      (effects (font (size 1.27 1.27)) (justify left))
-    )
     (pin "HUB_PRTCTL" bidirectional (at 81.28 132.715 180)
+      (effects (font (size 1.27 1.27)) (justify left))
+    )
+    (pin "SHOST_SSRXP" bidirectional (at 81.28 151.765 180)
+      (effects (font (size 1.27 1.27)) (justify left))
+    )
+    (pin "SHOST_SSRXN" bidirectional (at 81.28 154.305 180)
       (effects (font (size 1.27 1.27)) (justify left))
     )
@@
       (effects (font (size 1.27 1.27)) (justify right))
     )
+    (pin "SSTXP" bidirectional (at 40.64 146.05 0)
+      (effects (font (size 1.27 1.27)) (justify right))
+    )
+    (pin "SSTXN" bidirectional (at 40.64 148.59 0)
+      (effects (font (size 1.27 1.27)) (justify right))
+    )
     (pin "SSRXN" bidirectional (at 40.64 154.305 0)
       (effects (font (size 1.27 1.27)) (justify right))
     )
-    (pin "SSTXP" bidirectional (at 40.64 146.05 0)
-      (effects (font (size 1.27 1.27)) (justify right))
-    )
     (pin "SSRXP" bidirectional (at 40.64 151.765 0)
       (effects (font (size 1.27 1.27)) (justify right))
     )
-    (pin "SSTXN" bidirectional (at 40.64 148.59 0)
-      (effects (font (size 1.27 1.27)) (justify right))
-    )

Commit message: Almost ready 2.0.0
Parts:
- C10: footprint Capacitor_SMD:C_0603_1608Metric_Pad1.08x0.95mm_HandSolder -> Capacitor_SMD:C_0603_1608Metric; MFN (none) -> CL10A225KP8NNNC; MPN (none) -> CL10A225KP8NNNC
- C14, C15, C16, C17, C18, C7, C74, C76: MFN (none) -> CL10B104KB8NNNC
- C66, C67: MFN (none) -> CC0402JRNPO9BN120; MPN (none) -> CC0402JRNPO9BN120
- C73, C75: footprint Capacitor_SMD:C_0603_1608Metric_Pad1.08x0.95mm_HandSolder -> Capacitor_SMD:C_0603_1608Metric; MFN (none) -> CL10B105KA8NNNC; MPN (none) -> CL10B105KA8NNNC
- D1: Link (none) -> https://eu.mouser.com/ProductDetail/onsemi-Fairchild/1N4148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; MFN (none) -> 1N4148WT; MPN (none) -> 1N4148WT
- D2, D3, D4, D5: MFN (none) -> LTST-C190KRKT; MPN (none) -> LTST-C190KRKT
- J20: MFN (none) -> A2541WV-2X5P
- J21: MFN (none) -> A2541WV-2X3P
- J28: value CASE CONNECTORS -> 6x2 2.54mm header; MFN (none) -> A2541WV-2X3P; MPN (none) -> A2541WV-2X3P
- R1, R2: MFN (none) -> RC0402JR-0750RL; MPN (none) -> RC0402JR-0750RL
- R10: value 4k7 -> 10k; MFN (none) -> RTT02103JTH; MPN (none) -> RTT02103JTH
- R109, R110, R111, R112, R16, R20, R21, R23: MFN (none) -> RTT02471JTH; MPN (none) -> RTT02471JTH
- R15, R22: MFN (none) -> RTT02103JTH; MPN (none) -> RTT02103JTH
- SW1, SW2: MFN (none) -> K2-1102BQ-C4CW-01; MPN (none) -> K2-1102BQ-C4CW-01
- SW3: MFN (none) -> K2-1102SP-C4SC-04; MPN (none) -> K2-1102SP-C4SC-04
- U1: MFN (none) -> STM32F411CEU6; MPN (none) -> STM32F411CEU6
- Y1: MFN (none) -> SX32Y025000BG1T
