File: hardware/power_supplies.kicad_sch (KiCad schematic)
At the start: 43 parts, among them J23 DNM, J6 Conn_01x03_Pin, J6 Molex 4 Pin Peripheral Power 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, U3 AP2127N-3.3, U9 MIC23201YML

Commit message: Almost ready 2.0.0
Parts:
- C1, C2, C4, C79: footprint Capacitor_SMD:C_0603_1608Metric_Pad1.08x0.95mm_HandSolder -> Capacitor_SMD:C_0603_1608Metric; MFN (none) -> CL10B105KA8NNNC; MPN (none) -> CL10B105KA8NNNC
- C77, C78: MFN (none) -> HV470M035E055ETR; MPN (none) -> HV470M035E055ETR
- C80, C? (x6): MFN (none) -> CL10B104KB8NNNC
- C? (x2): MFN (none) -> CL05B471KB5NNNC; MPN (none) -> CL05B471KB5NNNC
- C? (x4): footprint Capacitor_SMD:C_0603_1608Metric_Pad1.08x0.95mm_HandSolder -> Capacitor_SMD:C_0603_1608Metric; MFN (none) -> C1608X5R1A226MT000E; MPN (none) -> C1608X5R1A226MT000E
- C? (x2): footprint Capacitor_SMD:C_0603_1608Metric_Pad1.08x0.95mm_HandSolder -> Capacitor_SMD:C_0603_1608Metric; MFN (none) -> CL10A225KP8NNNC; MPN (none) -> CL10A225KP8NNNC
- J6: MPN (none) -> 350211-1
- J6: MFN (none) -> PZ254V-11-03P
- L1, L3: MFN (none) -> MCL2012H100MT; MPN (none) -> MCL2012H100MT
- L2: MFN (none) -> LQH5BPN1R5NT0L
- L4: Link (none) -> https://www2.mouser.com/ProductDetail/Wurth-Elektronik/7427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; MFN (none) -> 7427932; MPN (none) -> 7427932
- R? (x5): MFN (none) -> RTT02103JTH; MPN (none) -> RTT02103JTH
- R?: value 5k1 -> 5k1 1%; MFN (none) -> RTT025101FTH; MPN (none) -> RTT025101FTH
- R?: value 12k -> 12k 1%; MFN (none) -> RTT021202FTH; MPN (none) -> RTT021202FTH
- R?: value 22k -> 22k 1%; MFN (none) -> CR0402FF2202G; MPN (none) -> CR0402FF2202G
- U3: Link (none) -> https://www.mouser.es/ProductDetail/Diodes-Incorporated/AP2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; MFN (none) -> AP2127N-3.3TRG1; MPN (none) -> AP2127N-3.3TRG1
- U9: Link (none) -> https://www2.mouser.com/ProductDetail/Microchip-Technology/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; MFN (none) -> MIC23201YML-TR; MPN (none) -> MIC23201YML-TR
