File: dutlink.kicad_pcb (KiCad board)
At the start: 4 copper layers, 170 x 170 mm, 142 parts, among them J1 USB_C_Receptacle_PowerOnly_6P, J10 I2C connector, J11 SPI/TPM connector, J16 Conn_01x02_Pin, J17 6x2 2.54mm header, J2 Barrel_Jack_MountingPin, J3 Barrel_Jack_MountingPin, J4 Conn_01x09_Pin, J5 USB_C_Receptacle_PowerOnly_6P, J6 Conn_01x05_Pin, J7 USB3_B, J8 Hirose USB3_B_Micro, J9 USB3_A, P1 USB_C_Plug_USB2.0, Q1 FDC6330L, Q2 FDC6330L, Q3 FDC6330L, Q4 FDC6330L, SW1 SW_Push, SW2 SW_Push, SW3 SW_Push, U1 STM32F411CEUx, U2 AP2127N-3.3, U3 AP2127N-3.3, U4 ACS725LLCTR-05AB-T, U6 TMUXHS4212, Y2 25 Mhz Crystal

Commit message: Reorganized repo with rename to dutlink 1.1.0
Signed-off-by: Miguel Angel Ajo Pelayo <majopela@redhat.com>
Parts:
- added C28: 100nF, Capacitor_SMD:C_0603_1608Metric, F.Cu at (177.5, 75.6)
- added R40: 330, Resistor_SMD:R_0402_1005Metric, F.Cu at (178.8, 75.6)
- C1, C10, C11, C12, C13, C14, C15, C17, C18, C2, C3, C31, C32, C4, C6, C8, C9: footprint Capacitor_SMD:C_0603_1608Metric_Pad1.08x0.95mm_HandSolder -> Capacitor_SMD:C_0603_1608Metric
- C19, C20, C21, C22, C24, C26, C33, C34, C35, C36, C37: footprint Capacitor_SMD:C_0402_1005Metric -> Capacitor_SMD:C_0603_1608Metric
- R35, R36, R37, R38, R39: footprint Resistor_SMD:R_0402_1005Metric -> Resistor_SMD:R_0603_1608Metric
- U5: value ~ -> TMUXHS221NKGR
- moved C21 2.19 mm to (100.8, 191.6)
- moved C20 1.66 mm to (121.2, 203.0)
- moved C19 1.16 mm to (121.2, 201.4)
- moved C22 0.87 mm to (102.3, 189.9)
- moved C37 0.47 mm to (70.6, 208.0)
- moved R39 0.24 mm to (102.3, 203.8)
- moved C34 0.16 mm to (114.7, 212.9)
Connections:
- P1 pad S1: GND -> Net-(P1-SHIELD)
Routing:
- net Net-(P1-SHIELD): track 0.00 -> 29.4 mm
- net GND: track 112.5 -> 118.2 mm, vias 87 -> 89
- net /USB_PW_HOST: track 141.9 -> 138.8 mm
- net VCC: track 96.7 -> 99.2 mm, vias 6 -> 8
- net +5V: track 32.5 -> 34.2 mm
- net GNDA: track 117.5 -> 119.1 mm
- net /ON_OFF: track 99.4 -> 100.9 mm
- net /board_control/VCCOUT: track 264.4 -> 262.9 mm
- net +3.3VA: track 122.7 -> 123.6 mm
- net Net-(J5-SHIELD): track 21.8 -> 22.7 mm
- net Net-(J9-SHIELD): track 40.3 -> 40.9 mm
- net /USB_STORAGE_MUX/VBUS_DUT: track 89.3 -> 88.7 mm
- added copper zone on F.Cu, net /board_control/VCCOUT
- added copper zone on F.Cu, net /board_control/VCCOUT_SW
- added copper zone on B.Cu, net VCC
Other:
- board text added: "NEVER CONNECT BOTH"

Commit message: 2.0.0 release
Parts:
- removed 3v3, 5V1: TestPoint, TestPoint:TestPoint_Pad_D1.0mm
- removed J11: SPI/TPM connector, Connector_PinHeader_2.54mm:PinHeader_2x05_P2.54mm_Vertical
- removed P1: USB_C_Plug_USB2.0, Connector_USB:USB_C_Receptacle_G-Switch_GT-USB-7010ASV
- removed the REF** at (91.5, 202.2)
- removed the REF** at (65.2, 105.9)
- removed the REF** at (75.1, 106.3)
- removed the REF** at (75.3, 93.5)
- removed the REF** at (148.6, 65.0)
- removed U2: AP2127N-3.3, Package_TO_SOT_SMD:SOT-23
- added 3v1: TestPoint, TestPoint:TestPoint_Pad_D1.0mm, F.Cu at (77.8, 107.0)
- added C100: 100nF, Capacitor_SMD:C_0402_1005Metric, F.Cu at (131.0, 183.2)
- added C101: 100nF, Capacitor_SMD:C_0402_1005Metric, F.Cu at (99.4, 79.4)
- added C102: 100nF, Capacitor_SMD:C_0402_1005Metric, F.Cu at (117.5, 136.9)
- added C103: 100nF, Capacitor_SMD:C_0402_1005Metric, F.Cu at (127.8, 101.5)
- added C104: 100nF, Capacitor_SMD:C_0402_1005Metric, F.Cu at (97.5, 101.5)
- added C105: 100nF, Capacitor_SMD:C_0402_1005Metric, F.Cu at (158.6, 101.6)
- added C39: 100nF, Capacitor_SMD:C_0402_1005Metric, F.Cu at (137.3, 148.0)
- added C40: 100nF, Capacitor_SMD:C_0402_1005Metric, F.Cu at (118.1, 146.2)
- added C41: 100nF, Capacitor_SMD:C_0402_1005Metric, F.Cu at (129.3, 135.3)
- added C42: 100nF, Capacitor_SMD:C_0402_1005Metric, F.Cu at (137.3, 148.9)
- added C43: 100nF, Capacitor_SMD:C_0402_1005Metric, F.Cu at (137.2, 145.3)
- added C44: 100nF, Capacitor_SMD:C_0402_1005Metric, F.Cu at (137.2, 143.0)
- added C45: 100nF, Capacitor_SMD:C_0402_1005Metric, F.Cu at (121.5, 152.9)
- added C46: 100nF, Capacitor_SMD:C_0402_1005Metric, F.Cu at (121.5, 152.0)
- added C47: 100nF, Capacitor_SMD:C_0402_1005Metric, F.Cu at (130.9, 153.2)
- added C48: 100nF, Capacitor_SMD:C_0402_1005Metric, F.Cu at (122.2, 136.3)
- added C49: 100nF, Capacitor_SMD:C_0402_1005Metric, F.Cu at (127.8, 135.3)
- added C50: 100nF, Capacitor_SMD:C_0402_1005Metric, F.Cu at (131.3, 135.3)
- added C51: 100nF, Capacitor_SMD:C_0402_1005Metric, F.Cu at (110.2, 80.6)
- added C52: 100nF, Capacitor_SMD:C_0402_1005Metric, F.Cu at (111.2, 80.6)
- added C53: 100nF, Capacitor_SMD:C_0402_1005Metric, F.Cu at (135.4, 102.0)
- added C54: 100nF, Capacitor_SMD:C_0402_1005Metric, F.Cu at (136.4, 102.0)
- added C55: 100nF, Capacitor_SMD:C_0402_1005Metric, F.Cu at (104.7, 102.2)
- added C56: 100nF, Capacitor_SMD:C_0402_1005Metric, F.Cu at (105.6, 102.2)
- added C57: 100nF, Capacitor_SMD:C_0402_1005Metric, F.Cu at (166.2, 102.0)
- added C58: 100nF, Capacitor_SMD:C_0402_1005Metric, F.Cu at (167.1, 102.0)
- added C59: 22uF, Capacitor_SMD:C_0603_1608Metric, F.Cu at (158.4, 132.9)
- added C60: 2.2uF, Capacitor_SMD:C_0603_1608Metric, F.Cu at (159.9, 132.9)
- added C61: 100nF, Capacitor_SMD:C_0402_1005Metric, F.Cu at (146.1, 67.5)
- added C62: 100nF, Capacitor_SMD:C_0402_1005Metric, F.Cu at (100.3, 210.9)
- added C63: 470pF, Capacitor_SMD:C_0402_1005Metric, F.Cu at (155.5, 135.8)
- added C64: 100nF, Capacitor_SMD:C_0402_1005Metric, F.Cu at (148.7, 134.3)
- added C65: 22uF, Capacitor_SMD:C_0603_1608Metric, F.Cu at (152.1, 128.7)
- added C66: 12pF, Capacitor_SMD:C_0402_1005Metric, F.Cu at (208.1, 154.9)
- added C67: 12pF, Capacitor_SMD:C_0402_1005Metric, F.Cu at (213.3, 155.0)
- added C68: 12pF, Capacitor_SMD:C_0402_1005Metric, F.Cu at (124.2, 131.9)
- added C69: 12pF, Capacitor_SMD:C_0402_1005Metric, F.Cu at (121.4, 134.4)
- added C70: 100nF, Capacitor_SMD:C_0402_1005Metric, F.Cu at (139.0, 170.4)
- added C71: 27pF, Capacitor_SMD:C_0402_1005Metric, F.Cu at (133.8, 175.5)
- added C72: 27pF, Capacitor_SMD:C_0402_1005Metric, F.Cu at (132.9, 180.8)
- added C73: 1uF, Capacitor_SMD:C_0603_1608Metric, F.Cu at (220.2, 160.3)
- added C74: 100nF, Capacitor_SMD:C_0402_1005Metric, F.Cu at (221.6, 160.1)
- added C75: 1uF, Capacitor_SMD:C_0603_1608Metric, F.Cu at (220.5, 120.4)
- added C76: 100nF, Capacitor_SMD:C_0402_1005Metric, F.Cu at (220.5, 121.6)
- added C77: 100nF, Capacitor_SMD:C_0402_1005Metric, F.Cu at (72.9, 94.0)
- added C78: 100nF, Capacitor_SMD:C_0402_1005Metric, F.Cu at (72.9, 95.2)
- added C79: 22uF, Capacitor_SMD:C_0603_1608Metric, F.Cu at (72.9, 96.8)
- added C80: 47uF 32V, Capacitor_SMD:CP_Elec_6.3x5.4_Nichicon, F.Cu at (82.5, 86.5)
- added C81: 47uF 32V, Capacitor_SMD:CP_Elec_6.3x5.4_Nichicon, F.Cu at (140.8, 88.1)
- added C82: 47uF 32V, Capacitor_SMD:CP_Elec_6.3x5.4_Nichicon, F.Cu at (92.6, 86.5)
- added C83: 1uF, Capacitor_SMD:C_0603_1608Metric, F.Cu at (77.8, 92.1)
- added C84: 100nF, Capacitor_SMD:C_0402_1005Metric, F.Cu at (80.0, 92.2)
- added C85: 2.2uF, Capacitor_SMD:C_0603_1608Metric, F.Cu at (73.3, 98.4)
- added C86: 470pF, Capacitor_SMD:C_0402_1005Metric, F.Cu at (76.1, 95.7)
- added C87: 100nF, Capacitor_SMD:C_0402_1005Metric, F.Cu at (78.1, 105.4)
- added C88: 22uF, Capacitor_SMD:C_0603_1608Metric, F.Cu at (77.9, 104.0)
- added C89: 4.7uF, Capacitor_SMD:C_0603_1608Metric, F.Cu at (129.6, 180.1)
- added C90: 100nF, Capacitor_SMD:C_0402_1005Metric, F.Cu at (144.3, 174.6)
- added C91: 100nF, Capacitor_SMD:C_0402_1005Metric, F.Cu at (133.8, 183.9)
- added C92: 100nF, Capacitor_SMD:C_0402_1005Metric, F.Cu at (138.1, 174.7)
- added C93: 100nF, Capacitor_SMD:C_0402_1005Metric, F.Cu at (150.1, 183.9)
- added C94: 100nF, Capacitor_SMD:C_0402_1005Metric, F.Cu at (142.6, 174.7)
- added C95: 100nF, Capacitor_SMD:C_0402_1005Metric, F.Cu at (139.5, 189.4)
- added C96: 100nF, Capacitor_SMD:C_0402_1005Metric, F.Cu at (145.2, 189.5)
- added C97: 100nF, Capacitor_SMD:C_0402_1005Metric, F.Cu at (149.6, 181.4)
- added C98: 100nF, Capacitor_SMD:C_0402_1005Metric, F.Cu at (131.0, 180.8)
- added C99: 4.7uF, Capacitor_SMD:C_0603_1608Metric, F.Cu at (129.6, 183.9)
- added D10: 1N4148WT, Diode_SMD:D_SOD-523, F.Cu at (117.6, 138.2)
- added D11: 1N4448WT, Diode_SMD:D_SOD-523, F.Cu at (86.9, 198.1)
- added D7: 1N4448WT, Diode_SMD:D_SOD-523, F.Cu at (142.0, 101.4)
- added D8: 1N4448WT, Diode_SMD:D_SOD-523, F.Cu at (110.5, 100.9)
- added D9: 1N4448WT, Diode_SMD:D_SOD-523, F.Cu at (172.6, 100.4)
- added F1: MF-MSMF125-2, FOOTPRINTS:MF-MSMF125-2, F.Cu at (144.8, 97.0)
- added F2: MF-MSMF125-2, FOOTPRINTS:MF-MSMF125-2, F.Cu at (114.1, 96.5)
- added F3: MF-MSMF125-2, FOOTPRINTS:MF-MSMF125-2, F.Cu at (176.3, 96.2)
- added F4: MF-MSMF125-2, FOOTPRINTS:MF-MSMF125-2, F.Cu at (70.8, 217.3)
- added FID1: Fiducial, Fiducial:Fiducial_0.5mm_Mask1mm, F.Cu at (60.0, 66.6)
- added FID2: Fiducial, Fiducial:Fiducial_0.5mm_Mask1mm, F.Cu at (127.9, 107.6)
- added FID3: Fiducial, Fiducial:Fiducial_0.5mm_Mask1mm, F.Cu at (211.8, 225.0)
- added FID4: Fiducial, Fiducial:Fiducial_0.5mm_Mask1mm, F.Cu at (150.3, 169.4)
- added FID5: Fiducial, Fiducial:Fiducial_0.5mm_Mask1mm, F.Cu at (226.1, 73.7)
- added FID6: Fiducial, Fiducial:Fiducial_0.5mm_Mask1mm, F.Cu at (117.1, 165.7)
- added GNDA1: TestPoint, TestPoint:TestPoint_Pad_D1.0mm, F.Cu at (158.0, 85.9)
- added H16: Board MountingHole, MountingHole:MountingHole_2.7mm_M2.5_Pad_Via, F.Cu at (208.3, 196.2)
- added J18: USB3_A, Connector_USB:SS-52000-004, F.Cu at (108.7, 97.1)
- added J19: USB3_A, Connector_USB:SS-52000-004, F.Cu at (170.2, 96.9)
- added J20: SPI/TPM connector, Connector_PinHeader_2.54mm:PinHeader_2x05_P2.54mm_Vertical, F.Cu at (219.3, 124.4)
- added J21: I2C connector, Connector_PinHeader_2.54mm:PinHeader_2x03_P2.54mm_Vertical, F.Cu at (219.3, 163.8)
- added J22: NC, Connector:Tag-Connect_TC2050-IDC-FP_2x05_P1.27mm_Vertical, F.Cu at (207.6, 135.6)
- added J23: DNM, Connector_BarrelJack:BarrelJack_Horizontal, F.Cu at (94.4, 75.1)
- added J24: Conn_01x03_Pin, Connector_PinHeader_2.54mm:PinHeader_1x03_P2.54mm_Vertical, F.Cu at (73.4, 73.0)
- added J27: Conn_02x20_Odd_Even, Connector_PinHeader_2.54mm:PinHeader_2x20_P2.54mm_Vertical_SMD, F.Cu at (158.1, 213.5)
- added J28: 6x2 2.54mm header, Connector_PinHeader_2.54mm:PinHeader_2x06_P2.54mm_Vertical, F.Cu at (219.3, 205.9)
- added L5: 7427932, FOOTPRINTS:7427932, F.Cu at (129.2, 86.2)
- added L6: 1.5uH, FOOTPRINTS:LQH5BPB100MT0L, F.Cu at (83.1, 103.1)
- added L7: 120Ω@100MH, Inductor_SMD:L_0402_1005Metric, F.Cu at (127.8, 182.7)
- added L8: 120Ω@100MH, Inductor_SMD:L_0402_1005Metric, F.Cu at (127.8, 181.2)
- added R100: 100, Resistor_SMD:R_0402_1005Metric, F.Cu at (170.3, 199.8)
- added R101: 100, Resistor_SMD:R_0402_1005Metric, F.Cu at (173.3, 206.6)
- added R102: 100, Resistor_SMD:R_0402_1005Metric, F.Cu at (173.0, 199.8)
- added R103: 100, Resistor_SMD:R_0402_1005Metric, F.Cu at (175.8, 206.6)
- added R104: 100, Resistor_SMD:R_0402_1005Metric, F.Cu at (175.6, 199.8)
- added R105: 100, Resistor_SMD:R_0402_1005Metric, F.Cu at (180.9, 206.6)
- added R106: 100, Resistor_SMD:R_0402_1005Metric, F.Cu at (180.6, 199.8)
- added R107: NC, Resistor_SMD:R_0805_2012Metric_Pad1.20x1.40mm_HandSolder, F.Cu at (130.0, 202.8)
- added R108: NC, Resistor_SMD:R_0805_2012Metric_Pad1.20x1.40mm_HandSolder, F.Cu at (155.4, 203.2)
- added R109: 470, Resistor_SMD:R_0402_1005Metric, F.Cu at (222.8, 192.1)
- added R110: 470, Resistor_SMD:R_0402_1005Metric, F.Cu at (220.2, 192.1)
- added R111: 470, Resistor_SMD:R_0402_1005Metric, F.Cu at (217.7, 192.1)
- added R112: 470, Resistor_SMD:R_0402_1005Metric, F.Cu at (215.1, 192.1)
- added R113: 2k, Resistor_SMD:R_0402_1005Metric, F.Cu at (104.5, 192.7)
- added R114: 330, Resistor_SMD:R_0402_1005Metric, F.Cu at (71.4, 208.8)
- added R115: 330, Resistor_SMD:R_0402_1005Metric, F.Cu at (130.2, 210.7)
- added R116: 330, Resistor_SMD:R_0402_1005Metric, F.Cu at (146.2, 71.0)
- added R117: 330, Resistor_SMD:R_0402_1005Metric, F.Cu at (99.7, 213.2)
- added R118: NC 10k, Resistor_SMD:R_0402_1005Metric, F.Cu at (174.6, 196.8)
- added R41: 10k, Resistor_SMD:R_0402_1005Metric, F.Cu at (73.5, 99.9)
- added R42: 22k 1%, Resistor_SMD:R_0402_1005Metric, F.Cu at (81.2, 97.6)
- added R43: 5k1 1%, Resistor_SMD:R_0402_1005Metric, F.Cu at (81.2, 96.5)
- added R44: 10k, Resistor_SMD:R_0402_1005Metric, F.Cu at (142.3, 139.7)
- added R45: 10k, Resistor_SMD:R_0402_1005Metric, F.Cu at (139.8, 140.4)
- added R46: 10k, Resistor_SMD:R_0402_1005Metric, F.Cu at (142.3, 141.0)
- added R47: 10k, Resistor_SMD:R_0402_1005Metric, F.Cu at (139.8, 144.0)
- added R48: 10k, Resistor_SMD:R_0402_1005Metric, F.Cu at (142.3, 144.6)
- added R49: 10k, Resistor_SMD:R_0402_1005Metric, F.Cu at (139.8, 145.3)
- added R50: 12k 1%, Resistor_SMD:R_0402_1005Metric, F.Cu at (120.0, 136.9)
- added R51: 200K, Resistor_SMD:R_0402_1005Metric, F.Cu at (142.3, 142.1)
- added R52: 200K, Resistor_SMD:R_0402_1005Metric, F.Cu at (139.8, 141.6)
- added R53: 200K, Resistor_SMD:R_0402_1005Metric, F.Cu at (112.5, 149.5)
- added R54: 200K, Resistor_SMD:R_0402_1005Metric, F.Cu at (114.6, 148.9)
- added R55: 10k, Resistor_SMD:R_0402_1005Metric, F.Cu at (112.5, 148.4)
- added R56: 10k, Resistor_SMD:R_0402_1005Metric, F.Cu at (142.3, 143.3)
- added R57: 10k, Resistor_SMD:R_0402_1005Metric, F.Cu at (139.8, 139.2)
- added R58: 10k, Resistor_SMD:R_0402_1005Metric, F.Cu at (134.0, 135.3)
- added R59: 200K, Resistor_SMD:R_0402_1005Metric, F.Cu at (132.0, 154.0)
- added R60: 200K, Resistor_SMD:R_0402_1005Metric, F.Cu at (132.4, 156.1)
- added R61: 200K, Resistor_SMD:R_0402_1005Metric, F.Cu at (133.3, 154.0)
- added R62: 200K, Resistor_SMD:R_0402_1005Metric, F.Cu at (133.7, 156.1)
- added R63: 200K, Resistor_SMD:R_0402_1005Metric, F.Cu at (134.6, 154.0)
- added R64: NC 10k, Resistor_SMD:R_0402_1005Metric, F.Cu at (117.4, 140.6)
- added R65: 10k, Resistor_SMD:R_0402_1005Metric, F.Cu at (142.3, 145.8)
- added R66: 330, Resistor_SMD:R_0402_1005Metric, F.Cu at (100.6, 79.3)
- added R67: 10k, Resistor_SMD:R_0402_1005Metric, F.Cu at (117.5, 139.5)
- added R68: 330, Resistor_SMD:R_0402_1005Metric, F.Cu at (125.7, 101.5)
- added R69: 330, Resistor_SMD:R_0402_1005Metric, F.Cu at (95.4, 101.5)
- added R70: 330, Resistor_SMD:R_0402_1005Metric, F.Cu at (156.7, 101.6)
- added R71: 200K, Resistor_SMD:R_0402_1005Metric, F.Cu at (127.8, 157.6)
- added R72: 200K, Resistor_SMD:R_0402_1005Metric, F.Cu at (128.9, 157.6)
- added R73: 100, Resistor_SMD:R_0402_1005Metric, F.Cu at (132.7, 206.6)
- added R74: 100, Resistor_SMD:R_0402_1005Metric, F.Cu at (132.5, 199.8)
- added R75: 100, Resistor_SMD:R_0402_1005Metric, F.Cu at (135.3, 206.6)
- added R76: 100, Resistor_SMD:R_0402_1005Metric, F.Cu at (135.2, 199.8)
- added R77: 100, Resistor_SMD:R_0402_1005Metric, F.Cu at (137.8, 206.6)
- added R78: 100, Resistor_SMD:R_0402_1005Metric, F.Cu at (137.5, 199.8)
- added R79: 100, Resistor_SMD:R_0402_1005Metric, F.Cu at (140.2, 206.6)
- added R80: 100, Resistor_SMD:R_0402_1005Metric, F.Cu at (139.9, 199.8)
- added R81: 100, Resistor_SMD:R_0402_1005Metric, F.Cu at (142.9, 206.6)
- added R82: 100, Resistor_SMD:R_0402_1005Metric, F.Cu at (142.4, 199.8)
- added R83: 100, Resistor_SMD:R_0402_1005Metric, F.Cu at (145.3, 206.6)
- added R84: 100, Resistor_SMD:R_0402_1005Metric, F.Cu at (145.0, 199.8)
- added R85: 100, Resistor_SMD:R_0402_1005Metric, F.Cu at (147.9, 206.6)
- added R86: 100, Resistor_SMD:R_0402_1005Metric, F.Cu at (147.7, 199.8)
- added R87: 100, Resistor_SMD:R_0402_1005Metric, F.Cu at (150.4, 206.6)
- added R88: 100, Resistor_SMD:R_0402_1005Metric, F.Cu at (150.2, 199.8)
- added R89: 100, Resistor_SMD:R_0402_1005Metric, F.Cu at (158.2, 206.6)
- added R90: 100, Resistor_SMD:R_0402_1005Metric, F.Cu at (158.0, 199.8)
- added R91: 100, Resistor_SMD:R_0402_1005Metric, F.Cu at (160.6, 206.6)
- added R92: 100, Resistor_SMD:R_0402_1005Metric, F.Cu at (160.4, 199.8)
- added R93: 100, Resistor_SMD:R_0402_1005Metric, F.Cu at (163.2, 206.6)
- added R94: 100, Resistor_SMD:R_0402_1005Metric, F.Cu at (162.9, 199.8)
- added R95: 100, Resistor_SMD:R_0402_1005Metric, F.Cu at (165.6, 206.6)
- added R96: 100, Resistor_SMD:R_0402_1005Metric, F.Cu at (165.3, 199.8)
- added R97: 100, Resistor_SMD:R_0402_1005Metric, F.Cu at (168.2, 206.6)
- added R98: 100, Resistor_SMD:R_0402_1005Metric, F.Cu at (167.8, 199.8)
- added R99: 100, Resistor_SMD:R_0402_1005Metric, F.Cu at (170.7, 206.6)
- added REF**: Symbol_Barrel_Polarity, Symbol:Symbol_Barrel_Polarity, F.Cu at (91.1, 202.7)
- added REF**: OSHW-Logo2_14.6x12mm_SilkScreen, Symbol:OSHW-Logo2_14.6x12mm_SilkScreen, F.Cu at (203.7, 169.0)
- added REF**: WEEE-Logo_4.2x6mm_SilkScreen, Symbol:WEEE-Logo_4.2x6mm_SilkScreen, F.Cu at (222.7, 184.9)
- added REF**: Symbol_Barrel_Polarity, Symbol:Symbol_Barrel_Polarity, F.Cu at (163.4, 75.3)
- added TP1: TestPoint, TestPoint:TestPoint_Pad_D1.0mm, F.Cu at (195.1, 145.0)
- added TP14: TestPoint, TestPoint:TestPoint_Pad_D1.0mm, F.Cu at (118.0, 134.3)
- added TP2: TestPoint, TestPoint:TestPoint_Pad_D1.0mm, F.Cu at (192.2, 145.9)
- added TP5: TestPoint, TestPoint:TestPoint_Pad_D1.0mm, F.Cu at (216.6, 77.9)
- added TP6: TestPoint, TestPoint:TestPoint_Pad_D1.0mm, F.Cu at (163.6, 82.4)
- added TP8: TestPoint, TestPoint:TestPoint_Pad_D1.0mm, F.Cu at (148.2, 137.6)
- added U10: 93LC56BT-E/OT, Package_TO_SOT_SMD:SOT-23-6, F.Cu at (141.8, 171.5)
- added U11: MIC23201YML, FOOTPRINTS:SON50P300X300X100-11N-D, F.Cu at (77.5, 98.4)
- added U7: FT2232HQ, Package_DFN_QFN:QFN-64-1EP_9x9mm_P0.5mm_EP4.35x4.35mm, F.Cu at (141.8, 182.1)
- added U8: USB7206CT/KDX, VQFN100:VQFN100_KDX_MCH, F.Cu at (128.2, 144.4)
- added U9: MIC23201YML, FOOTPRINTS:SON50P300X300X100-11N-D, F.Cu at (153.5, 133.4)
- added Y1: 25 Mhz Crystal +/- 10ppm, Oscillator:Oscillator_SMD_EuroQuartz_XO32-4Pin_3.2x2.5mm, F.Cu at (210.7, 154.9)
- added Y3: Cristales 12.000 MHZ 10PF, Oscillator:Oscillator_SMD_EuroQuartz_XO32-4Pin_3.2x2.5mm, F.Cu at (133.7, 178.3)
- C13, C14, C15, C16, C17, C18, C20, C22, C24, C26, C28, C32, C33, C34, C35, C36, C37, C7: footprint Capacitor_SMD:C_0603_1608Metric -> Capacitor_SMD:C_0402_1005Metric
- C23, C25: value 1uF -> 100nF; footprint Capacitor_SMD:C_0603_1608Metric -> Capacitor_SMD:C_0402_1005Metric
- C27, C38: value 47uF 32V -> 100nF; footprint Capacitor_SMD:CP_Elec_6.3x5.4_Nichicon -> Capacitor_SMD:C_0402_1005Metric
- C3: value 1uF -> 3.3uF
- C8, C9: value 12pF -> 100nF; footprint Capacitor_SMD:C_0603_1608Metric -> Capacitor_SMD:C_0402_1005Metric
- J10: value I2C connector -> SPI/TPM connector; footprint Connector_PinHeader_2.54mm:PinHeader_2x03_P2.54mm_Vertical -> Connector_PinHeader_2.54mm:PinHeader_2x05_P2.54mm_Vertical
- J17: value 6x2 2.54mm header -> USB3_B; footprint Connector_PinHeader_2.54mm:PinHeader_2x06_P2.54mm_Vertical -> USB3Wurth:Wurth WR-COM USB 3.0 692221030100
- J6: value Conn_01x05_Pin -> Molex 4 Pin Peripheral Power Connector; footprint Connector_PinHeader_2.54mm:PinHeader_1x05_P2.54mm_Vertical -> FOOTPRINTS:3502111
- J7: value USB3_B -> USB3_A; footprint USB3Wurth:Wurth WR-COM USB 3.0 692221030100 -> Connector_USB:SS-52000-004
- L2: value 7427932 -> 1.5uH; footprint FOOTPRINTS:7427932 -> FOOTPRINTS:LQH5BPB100MT0L
- R1, R11, R12, R13, R14, R15, R2, R22, R24, R27, R28, R29, R3, R30, R31, R4, R5, R6, R7: footprint Resistor_SMD:R_0603_1608Metric -> Resistor_SMD:R_0402_1005Metric
- R10: value 4k7 -> 10k; footprint Resistor_SMD:R_0603_1608Metric -> Resistor_SMD:R_0402_1005Metric
- R16, R20, R21, R23: value 1k -> 470; footprint Resistor_SMD:R_0603_1608Metric -> Resistor_SMD:R_0402_1005Metric
- R17, R18, R33, R34, R40: value 330 -> 10k
- R19: value 5k1 -> 10k; footprint Resistor_SMD:R_0603_1608Metric -> Resistor_SMD:R_0402_1005Metric
- R25: value 0 -> 43K; footprint Resistor_SMD:R_0603_1608Metric -> Resistor_SMD:R_0402_1005Metric
- R26: value 0 -> 49K9 1%; footprint Resistor_SMD:R_0603_1608Metric -> Resistor_SMD:R_0402_1005Metric
- R32: value 330 -> 12k 1%
- R35, R39: value 470 -> 10k; footprint Resistor_SMD:R_0603_1608Metric -> Resistor_SMD:R_0402_1005Metric
- R36, R38: value 470 -> 2k; footprint Resistor_SMD:R_0603_1608Metric -> Resistor_SMD:R_0402_1005Metric
- R37: value 470 -> 12k 1%; footprint Resistor_SMD:R_0603_1608Metric -> Resistor_SMD:R_0402_1005Metric
- R8: value 2k4 -> 2k4 1%; footprint Resistor_SMD:R_0603_1608Metric -> Resistor_SMD:R_0402_1005Metric
- R9: value 470 -> 470 1%; footprint Resistor_SMD:R_0603_1608Metric -> Resistor_SMD:R_0402_1005Metric
- SW2: footprint Button_Switch_SMD:SW_SPST_B3S-1000 -> Button_Switch_THT:SW_Tactile_SPST_Angled_PTS645Vx58-2LFS
- U5: value TMUXHS221NKGR -> TMUXHS221
- Y2: value 25 Mhz Crystal -> 25 Mhz Crystal +/- 10ppm
- moved J17 171.8 mm to (107.3, 71.9), turned to 180 degrees
- moved C23 170.5 mm to (72.3, 208.7), turned to -90 degrees
- moved C28 164.9 mm to (80.5, 208.9), turned to 90 degrees
- moved REF** 156.8 mm to (63.8, 217.3)
- moved REF** 152.8 mm to (63.7, 206.1)
- moved C27 145.3 mm to (79.6, 208.9), turned to 90 degrees
- moved C25 135.3 mm to (125.8, 211.9)
- moved C26 134.1 mm to (126.7, 211.9), turned to 90 degrees
- moved J6 130.4 mm to (63.0, 86.0), turned to 90 degrees
- moved TP11 126.2 mm to (158.5, 88.4)
- moved C24 125.0 mm to (131.3, 210.7), turned to 90 degrees
- moved C3 112.3 mm to (145.6, 174.1), turned to 90 degrees
- moved R26 111.4 mm to (100.6, 81.5), turned to -90 degrees
- moved R40 102.5 mm to (78.4, 96.0), turned to 0 degrees
- moved R25 101.3 mm to (101.8, 81.5)
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Connections:
- C23 pad 1: GND -> Net-(J9-SHIELD)
- C23 pad 2: +3.3V -> GND
- C24 pad 1: +3.3V -> Net-(J8-SHIELD)
- C25 pad 1: GND -> /USB_STORAGE_MUX/DUT_SSRXN
- C25 pad 2: +3.3V -> /USB_STORAGE_MUX/_DUT_SSRXN
- C26 pad 1: +3.3V -> /USB_STORAGE_MUX/DUT_SSRXP
- C26 pad 2: GND -> /USB_STORAGE_MUX/_DUT_SSRXP
- C27 pad 1: VCC -> /USB_STORAGE_MUX/_STORAGE_SSTXN
- C27 pad 2: GND -> /USB_STORAGE_MUX/STORAGE_SSTXN
- C28 pad 1: Net-(P1-SHIELD) -> /USB_STORAGE_MUX/_STORAGE_SSTXP
- C28 pad 2: GND -> /USB_STORAGE_MUX/STORAGE_SSTXP
- C3 pad 1: +3.3V -> +1V8
- C33 pad 1: Net-(J1-SHIELD) -> VCORE
- C34 pad 1: Net-(J5-SHIELD) -> VCORE
- C35 pad 1: Net-(J7-SHIELD) -> VCORE
- C36 pad 1: Net-(J8-SHIELD) -> VCORE
- C37 pad 1: Net-(J9-SHIELD) -> VCORE
- C38 pad 1: /USB_STORAGE_MUX/VBUS_STORAGE -> VCORE
- C5 pad 1: VCC -> /board_control/_VCC
- C8 pad 1: GND -> +5V
- C8 pad 2: /XTALO -> GND
- C9 pad 1: GND -> +5V
- C9 pad 2: /XTALI -> GND
- J1 pad A9: /board_control/VCCIN -> /board_control/J1_VCC
- J1 pad B9: /board_control/VCCIN -> /board_control/J1_VCC
- J10 pad 1: +3.3V -> /board_control/J2_VCC
- J10 pad 2: /I2C1_SCL -> /board_control/_VCC
- J10 pad 3: GND -> /board_control/J1_VCC
- J10 pad 4: /I2C1_SDA -> /board_control/_VCC
- J10 pad 5: +3.3V -> /Power/12V_IN
- J10 pad 6: /IRQ_IN -> /board_control/_VCC
- J17 pad 1: Net-(J17-Pin_1) -> /Power/VBUS_UPSTREAM
- J17 pad 10: /BUTTON -> Net-(J17-SHIELD)
- J17 pad 2: +3.3V -> /USB 3.2 Gen2 front-hub/HOST_DN
- J17 pad 3: Net-(J17-Pin_3) -> /USB 3.2 Gen2 front-hub/HOST_DP
- J17 pad 4: +3.3V -> GND
- J17 pad 5: Net-(J17-Pin_5) -> /USB 3.2 Gen2 front-hub/HOST_SSTXN
- J17 pad 6: +3.3V -> /USB 3.2 Gen2 front-hub/HOST_SSTXP
- J17 pad 7: Net-(J17-Pin_7) -> GND
- J17 pad 8: +3.3V -> /USB 3.2 Gen2 front-hub/HOST_SSRXN
- J17 pad 9: GND -> /USB 3.2 Gen2 front-hub/HOST_SSRXP
- J2 pad 1: /board_control/VCCIN -> /board_control/J2_VCC
- J6 pad 1: +3.3V -> /Power/12V_IN
- J6 pad 2: /SWDIO -> GND
- J6 pad 3: /SWCLK -> GND
- J6 pad 4: GND -> /Power/5V_IN
- J7 pad 1: /USB_STORAGE_MUX/_VBUS_HOST -> Net-(D7-K)
- J7 pad 2: /USB_STORAGE_MUX/HOST_DN -> /USB 3.2 Gen2 front-hub/P1_DN
- J7 pad 3: /USB_STORAGE_MUX/HOST_DP -> /USB 3.2 Gen2 front-hub/P1_DP
- J7 pad 5: /USB_STORAGE_MUX/HOST_SSTXN -> /USB 3.2 Gen2 front-hub/P1_SSRXN
- J7 pad 6: /USB_STORAGE_MUX/HOST_SSTXP -> /USB 3.2 Gen2 front-hub/P1_SSRXP
- J7 pad 8: /USB_STORAGE_MUX/HOST_SSRXN -> /USB 3.2 Gen2 front-hub/P1_SSTXN
- J7 pad 9: /USB_STORAGE_MUX/HOST_SSRXP -> /USB 3.2 Gen2 front-hub/P1_SSTXP
- J9 pad 1: /USB_STORAGE_MUX/VBUS_STORAGE -> /USB_STORAGE_MUX/VBUS_STORAGE_
- L1 pad 1: +5VA -> GNDA
- L1 pad 2: +5V -> GND
- L2 pad 1: /board_control/VCCIN -> /Power/LVCORE
- L2 pad 2: VCC -> VCORE
- L3 pad 1: GNDA -> +5VA
- L3 pad 2: GND -> +5V
- L4 pad 1: /USB_STORAGE_MUX/_VBUS_HOST -> /Power/5V_IN_
- L4 pad 2: /USB_STORAGE_MUX/VBUS_HOST -> +5V
- Q3 pad 4: /USB_STORAGE_MUX/VBUS_HOST -> +5V
- R17 pad 1: GND -> VCORE
- R17 pad 2: Net-(J1-SHIELD) -> Net-(U9-PG)
- R18 pad 1: GND -> +5V
- R18 pad 2: Net-(J5-SHIELD) -> Net-(U9-EN)
- R19 pad 1: Net-(P1-CC1) -> VCORE
- R19 pad 2: GND -> /Power/FBVCORE
- R25 pad 1: Net-(U6-RSVD1) -> /USB 3.2 Gen2 front-hub/VBUS_MON_UP
- R25 pad 2: +3.3V -> /Power/VBUS_UPSTREAM
- R26 pad 1: Net-(U6-RSVD2) -> GND
- R26 pad 2: +3.3V -> /USB 3.2 Gen2 front-hub/VBUS_MON_UP
- R27 pad 1: /USB_STORAGE_MUX/VBUS_HOST -> +5V
- R32 pad 1: GND -> /Power/FBVCORE
- R32 pad 2: Net-(J7-SHIELD) -> GND
- R33 pad 1: GND -> +3.3V
- R33 pad 2: Net-(J8-SHIELD) -> /FT2232_EECS
- R34 pad 1: GND -> +3.3V
- R34 pad 2: Net-(J9-SHIELD) -> Net-(U10-DO)
- R35 pad 1: GND -> +3.3V
- R35 pad 2: Net-(J17-Pin_1) -> /FT2232_EECLK
- R36 pad 1: /LED2 -> Net-(U10-DO)
- R36 pad 2: Net-(J17-Pin_3) -> /FT2232_EEDATA
- R37 pad 1: /LED1 -> Net-(U7-REF)
- R37 pad 2: Net-(J17-Pin_5) -> GND
- R38 pad 1: /LED0 -> /nRESET_OUT
- R38 pad 2: Net-(J17-Pin_7) -> +3.3V
- R39 pad 1: GND -> Net-(U8-SPI_CLK/PF21)
- R39 pad 2: Net-(J16-Pin_1) -> GND
- R40 pad 1: GND -> +3.3V
- R40 pad 2: Net-(P1-SHIELD) -> Net-(U11-PG)
- U1 pad 13: unconnected-(U1-PA3-Pad13) -> /FT2232_EECLK
- U1 pad 19: unconnected-(U1-PB1-Pad19) -> /FT2232_EECS
- U1 pad 31: unconnected-(U1-PA10-Pad31) -> /FT2232_EEDATA
- U1 pad 32: /_DN -> /DN
- U1 pad 33: /_DP -> /DP
- U1 pad 5: /XTALO -> /XTALI
- U1 pad 6: /XTALI -> /XTALO
- U5 pad 4: /USB_STORAGE_MUX/HOST_DN -> /SHOST_DN
- U5 pad 5: /USB_STORAGE_MUX/HOST_DP -> /SHOST_DP
- U6 pad 1: Net-(U6-RSVD1) -> +3.3V
- U6 pad 10: Net-(U6-RSVD2) -> +3.3V
- U6 pad 14: /USB_STORAGE_MUX/DUT_SSRXN -> /USB_STORAGE_MUX/_DUT_SSRXN
- U6 pad 15: /USB_STORAGE_MUX/DUT_SSRXP -> /USB_STORAGE_MUX/_DUT_SSRXP
- U6 pad 16: /USB_STORAGE_MUX/HOST_SSTXN -> /SHOST_SSTXN
- U6 pad 17: /USB_STORAGE_MUX/HOST_SSTXP -> /SHOST_SSTXP
- U6 pad 18: /USB_STORAGE_MUX/HOST_SSRXN -> /SHOST_SSRXN
- U6 pad 19: /USB_STORAGE_MUX/HOST_SSRXP -> /SHOST_SSRXP
- U6 pad 3: /USB_STORAGE_MUX/STORAGE_SSTXP -> /USB_STORAGE_MUX/STORAGE_SSRXP
- U6 pad 4: /USB_STORAGE_MUX/STORAGE_SSTXN -> /USB_STORAGE_MUX/STORAGE_SSRXN
- U6 pad 7: /USB_STORAGE_MUX/STORAGE_SSRXP -> /USB_STORAGE_MUX/_STORAGE_SSTXP
- U6 pad 8: /USB_STORAGE_MUX/STORAGE_SSRXN -> /USB_STORAGE_MUX/_STORAGE_SSTXN
- Y2 pad 1: /XTALO -> /USB 3.2 Gen2 front-hub/XTALO
- Y2 pad 3: /XTALI -> /USB 3.2 Gen2 front-hub/XTALI
Routing:
- net +3.3V: track 663.4 -> 152.4 mm, vias 18 -> 57
- net +5V: track 34.2 -> 254.2 mm, vias 3 -> 4
- net /USB_STORAGE_MUX/HOST_DP: track 137.6 -> 0.00 mm, vias 3 -> 0
- net /USB_STORAGE_MUX/HOST_DN: track 135.4 -> 0.00 mm, vias 3 -> 0
- net GND: track 118.2 -> 241.6 mm, vias 89 -> 233
- net /FT2232_EECS: track 0.00 -> 120.8 mm, vias 0 -> 2
- net /USB_STORAGE_MUX/HOST_SSTXN: track 115.6 -> 0.00 mm, vias 1 -> 0
- net /USB_STORAGE_MUX/HOST_SSRXN: track 115.5 -> 0.00 mm, vias 1 -> 0
- net /USB_STORAGE_MUX/HOST_SSRXP: track 115.5 -> 0.00 mm, vias 1 -> 0
- net /USB_STORAGE_MUX/HOST_SSTXP: track 115.5 -> 0.00 mm, vias 1 -> 0
- net /FT2232_EECLK: track 0.00 -> 110.8 mm, vias 0 -> 2
- net /Power/5V_IN: track 0.00 -> 104.5 mm
- net /DN: track 0.00 -> 98.8 mm, vias 0 -> 2
- net GNDA: track 119.1 -> 20.5 mm, vias 16 -> 9
- net /DP: track 0.00 -> 98.6 mm, vias 0 -> 2
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- added copper zone on F.Cu, net +3.3V
- added copper zone on In1.Cu, net +3.3V
- added copper zone on F.Cu, net +5V
- added copper zone on F.Cu, net /Power/LVCORE
- added copper zone on F.Cu, net /Power/LVCORE3
- added copper zone on F.Cu, net /USB_STORAGE_MUX/VBUS_DUT
- added copper zone on F.Cu, net /board_control/_VCC
- added copper zone on F.Cu, net GND
- added copper zone on F.Cu, net VCORE
- added copper zone on In1.Cu, net VCORE
- removed copper zone on F.Cu, net /board_control/VCCOUT
- removed copper zone on F.Cu, net /board_control/VCCOUT_SW
- removed copper zone on In1.Cu, net GND
- removed copper zone on In1.Cu, net GNDA
- removed copper zone on B.Cu, net VCC
Other:
- board text added: "AC0"
- board text added: "AC1"
- board text added: "AC2"
- board text added: "AC3"
- board text added: "AC4"
- board text added: "AC5"
- board text added: "AC6"
- board text added: "AC7"
- board text added: "AD0/TCK TXD"
- board text added: "AD1/TDI RXD"
- board text added: "AD2/TDO RTS#"
- board text added: "AD3/TMS CTS#"
- board text added: "AD4"
- board text added: "AD5"
- board text added: "AD6"
- board text added: "AD7"
- board text added: "ATX 5V"
- board text added: "BC0"
- board text added: "BC1"
- board text added: "BC2"
- board text added: "BC3"
- board text added: "BC4"
- board text added: "BC5"
- board text added: "BC6"
- board text added: "BC7"
- board text added: "BD0/TXD"
- board text added: "BD1/RXD"
- board text added: "BD2/RTS#"
- board text added: "BD3/CTS#"
- board text added: "BD4/DTR#"
- board text added: "BD5/DSR#"
- board text added: "BD6"
- board text added: "BD7"
- board text added: "BUTTON"
- board text added: "CASE LEDS"
- board text added: "DUT POWER INPUT"
- board text added: "DUT PWR_IN"
- board text added: "DUT PWR_IN 5-25V"
- board text added: "DUT Power Input Jumper"
- board text added: "DUTLINK POWER INPUT"
- board text added: "DUT_ON LED"
- board text added: "FT2232HQ USB to JTAG/SWD/UART/I2C/SPI/BUS"
- board text added: "HOST J17"
- board text added: "I2C/ SENSORS"
- board text added: "J2 J1 12V ATX 5V ATX 5V ATX"
- board text added: "Jumpstarter and USB Power"
- board text added: "PWREN"
- board text added: "REL 2.0.0"
- board text added: "SUSPEND#"
- board text added: "USB 3.1 Gen 2 Hub"
- board text added: "USB P1"
- board text added: "USB P2"
- board text added: "USB P3"
- board text added: "USB P4"
- board text added: "USB P5"
- board text added: "USB P6"
- board text added: "USB PORTS for extension: * CAN BUS * JTAG/PROGRAMMERS * ETHERNET * VIDEO CAPTURE * ..."
- board text added: "USB3 to HOST"
- board text added: "USBPD OUT"
- board text added: "do not connect V/IO or 3v3 to the DUT, only provided to enable voltage translation."
- board text added: "github.com/jumpstarter-dev/dutlink-board"
- board text removed: "CASE CONNECTIONS"
- board text removed: "HOST USB"
- board text removed: "I2C"
- board text removed: "NEVER CONNECT BOTH"
- board text removed: "POWER INPUT"
- board text removed: "PWR_IN"
- board text removed: "PWR_IN 5-25V"
- board text removed: "REL 1.1.0"
- board text removed: "STORAGE TO HOST"
- board text removed: "USBPD_OUT 5-20V"
- board text removed: "do not connect V/IO to device under test, only provided to enable voltage translation boards."
- board text removed: "github.com/redhat-et/dutlink-board"
