File: dutlink.kicad_sch (KiCad schematic)
At the start: 66 parts, among them J10 Conn_01x02_Pin, J11 Conn_01x02_Pin, J12 Conn_01x02_Pin, J13 Conn_01x02_Pin, J14 Conn_01x02_Pin, J15 Conn_01x02_Pin, J6 Conn_01x05_Pin, P1 USB_C_Plug_USB2.0, SW1 SW_Push, SW2 SW_Push, SW3 SW_Push, U1 STM32F411CEUx, U2 AP2127N-3.3, U3 AP2127N-3.3, Y2 25 Mhz Crystal

Commit message: Reorganized repo with rename to dutlink 1.1.0
Signed-off-by: Miguel Angel Ajo Pelayo <majopela@redhat.com>
Parts:
- removed GNDA1, TP1, TP2, TP3, TP4, TP5, TP6, TP7, TP9: TestPoint, TestPoint:TestPoint_Pad_D1.0mm, symbol Connector:TestPoint
- removed H17, H18: cable strap hole, MountingHole:MountingHole_4.3mm_M4_Pad_Via, symbol Mechanical:MountingHole
- removed J10, J11, J12, J13, J14, J15: Conn_01x02_Pin, Connector_PinHeader_2.54mm:PinHeader_1x02_P2.54mm_Vertical, symbol Connector:Conn_01x02_Pin
- removed R17, R18: 10, Resistor_SMD:R_0603_1608Metric, symbol Device:R
- added C23, C25: 1uF, Capacitor_SMD:C_0603_1608Metric, symbol Device:C
- added C24, C26, C28: 100nF, Capacitor_SMD:C_0603_1608Metric, symbol Device:C
- added J10: I2C connector, Connector_PinHeader_2.54mm:PinHeader_2x03_P2.54mm_Vertical, symbol Connector_Generic:Conn_02x03_Odd_Even
- added J11: SPI/TPM connector, Connector_PinHeader_2.54mm:PinHeader_2x05_P2.54mm_Vertical, symbol Connector_Generic:Conn_02x05_Odd_Even
- added J17: 6x2 2.54mm header, Connector_PinHeader_2.54mm:PinHeader_2x06_P2.54mm_Vertical, symbol Connector_Generic:Conn_02x06_Odd_Even
- added R35, R36, R37, R38: 470, Resistor_SMD:R_0603_1608Metric, symbol Device:R
- added R40: 330, Resistor_SMD:R_0402_1005Metric, symbol Device:R
- C1, C2, C3, C4: footprint Capacitor_SMD:C_0603_1608Metric_Pad1.08x0.95mm_HandSolder -> Capacitor_SMD:C_0603_1608Metric; MFN (none) -> CL10B105KA8NNNC
- C10: footprint Capacitor_SMD:C_0603_1608Metric_Pad1.08x0.95mm_HandSolder -> Capacitor_SMD:C_0603_1608Metric; MFN (none) -> CL10A225KP8NNNC
- C14, C15, C17, C18: footprint Capacitor_SMD:C_0603_1608Metric_Pad1.08x0.95mm_HandSolder -> Capacitor_SMD:C_0603_1608Metric; MFN (none) -> CL10B104KB8NNNC
- C16, C7: MFN (none) -> CL10B104KB8NNNC
- C8, C9: footprint Capacitor_SMD:C_0603_1608Metric_Pad1.08x0.95mm_HandSolder -> Capacitor_SMD:C_0603_1608Metric; MFN (none) -> CC0603JRNPO9BN120
- D1: MFN (none) -> 1N4148WT
- D2, D3, D4, D5: MFN (none) -> LTST-C190KRKT
- J6: MFN (none) -> B-2100S05P-A110
- L1, L3: MFN (none) -> MCL2012H100MT
- P1: symbol Connector:USB_C_Plug_USB2.0 -> Connector:USB_C_Receptacle_USB2.0; MFN (none) -> GT-USB-7010ASV
- R1, R2: MFN (none) -> RT0603BRE0750RL
- R10: MFN (none) -> RTT034701FTP
- R15, R22: MFN (none) -> CRCW060310K0FKEA
- R16, R20, R21, R23: MFN (none) -> RTT031001FTP
- R19: MFN (none) -> RC0603FR-075K1L
- SW1: MFN (none) -> K2-1102BQ-C4CW-01
- SW2, SW3: MFN (none) -> K2-1102SP-C4SC-04
- U1: MFN (none) -> STM32F411CEU6
- U2, U3: Link (none) -> https://www.mouser.es/ProductDetail/Diodes-Incorporated/AP2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; MFN (none) -> AP2127N-3.3TRG1
- Y2: MFN (none) -> SX32Y025000BG1T
Connections:
- net DN is gone; now on net _DN: U1.32 (PA11)
- net DP is gone; now on net _DP: U1.33 (PA12)
- net +3.3V: now also C23.2, C24.1, C25.2, C26.1, J10.1 (Pin_1), J10.5 (Pin_5), J11.1 (Pin_1), J17.2 (Pin_2), J17.4 (Pin_4), J17.6 (Pin_6), J17.8 (Pin_8)
- net BUTTON: now also J17.10 (Pin_10)
- net GND: now also C23.1, C24.2, C25.1, C26.2, C28.2, J10.3 (Pin_3), J11.4 (Pin_4), J11.9 (Pin_9), J17.11 (Pin_11), J17.9 (Pin_9), R35.1, R40.1; no longer C14.2, P1.S1 (SHIELD)
- net GNDA: now also C14.2
- net LED0: now also R38.1
- net LED1: now also R37.1
- net LED2: now also R36.1
- net NRST: now also J17.12 (Pin_12)
- net _DN: now also P1.B7 (D-)
- net _DP: now also P1.B6 (D+)
- net nRESET_OUT: now reaches U1.18 (PB0)
- net nRESET_OUT: now also J11.2 (Pin_2)
- net IRQ_IN: now reaches U1.21 (PB10)
- net IRQ_IN: now also J10.6 (Pin_6), J11.6 (Pin_6)
- net SPI2_NSS: now reaches U1.25 (PB12)
- net SPI2_NSS: now also J11.10 (Pin_10)
- net SPI2_SCK: now reaches U1.26 (PB13)
- net SPI2_SCK: now also J11.7 (Pin_7)
- net SPI2_MISO: now reaches U1.27 (PB14)
- net SPI2_MISO: now also J11.5 (Pin_5)
- net SPI2_MOSI: now reaches U1.28 (PB15)
- net SPI2_MOSI: now also J11.3 (Pin_3)
- net I2C1_SCL: now reaches U1.45 (PB8)
- net I2C1_SCL: now also J10.2 (Pin_2)
- net I2C1_SDA: now reaches U1.46 (PB9)
- net I2C1_SDA: now also J10.4 (Pin_4)
- new net: C28.1, P1.S1 (SHIELD), R40.2
- new net: J17.3 (Pin_3), R36.2
- new net: J17.1 (Pin_1), R35.2
- new net: J17.5 (Pin_5), R37.2
- new net: J17.7 (Pin_7), R38.2
- no-connect marks 0 -> 1
Other:
- moved on the sheet: 3v3, 3v3A1, 5V1, C1, C10, C14, C15, C16, C17, C18, C2, C3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

Commit message: 2.0.0 release
Parts:
- removed 3v3, 3v3A1, 5V1: TestPoint, TestPoint:TestPoint_Pad_D1.0mm, symbol Connector:TestPoint
- removed C1, C2, C23, C25, C3, C4: 1uF, Capacitor_SMD:C_0603_1608Metric, symbol Device:C
- removed C24, C26, C28: 100nF, Capacitor_SMD:C_0603_1608Metric, symbol Device:C
- removed C8, C9: 12pF, Capacitor_SMD:C_0603_1608Metric, symbol Device:C
- removed J10: I2C connector, Connector_PinHeader_2.54mm:PinHeader_2x03_P2.54mm_Vertical, symbol Connector_Generic:Conn_02x03_Odd_Even
- removed J11: SPI/TPM connector, Connector_PinHeader_2.54mm:PinHeader_2x05_P2.54mm_Vertical, symbol Connector_Generic:Conn_02x05_Odd_Even
- removed J17: 6x2 2.54mm header, Connector_PinHeader_2.54mm:PinHeader_2x06_P2.54mm_Vertical, symbol Connector_Generic:Conn_02x06_Odd_Even
- removed J6: Conn_01x05_Pin, Connector_PinHeader_2.54mm:PinHeader_1x05_P2.54mm_Vertical, symbol Connector:Conn_01x05_Pin
- removed L1, L3: 10uH, Inductor_SMD:L_0805_2012Metric, symbol Device:L_Ferrite
- removed P1: USB_C_Plug_USB2.0, Connector_USB:USB_C_Receptacle_G-Switch_GT-USB-7010ASV, symbol Connector:USB_C_Receptacle_USB2.0
- removed R19: 5k1, Resistor_SMD:R_0603_1608Metric, symbol Device:R
- removed R35, R36, R37, R38: 470, Resistor_SMD:R_0603_1608Metric, symbol Device:R
- removed R40: 330, Resistor_SMD:R_0402_1005Metric, symbol Device:R
- removed U2, U3: AP2127N-3.3, Package_TO_SOT_SMD:SOT-23, symbol Regulator_Linear:AP2127N-3.3
- removed Y2: 25 Mhz Crystal, Oscillator:Oscillator_SMD_EuroQuartz_XO32-4Pin_3.2x2.5mm, symbol Device:Crystal_GND24
- added C66, C67: 12pF, Capacitor_SMD:C_0402_1005Metric, symbol Device:C
- added C73, C75: 1uF, Capacitor_SMD:C_0603_1608Metric, symbol Device:C
- added C74, C76: 100nF, Capacitor_SMD:C_0402_1005Metric, symbol Device:C
- added FID1, FID2, FID3, FID4, FID5, FID6: Fiducial, Fiducial:Fiducial_0.5mm_Mask1mm, symbol Mechanical:Fiducial
- added GNDA1, TP1, TP2, TP5, TP6: TestPoint, TestPoint:TestPoint_Pad_D1.0mm, symbol Connector:TestPoint
- added J20: SPI/TPM connector, Connector_PinHeader_2.54mm:PinHeader_2x05_P2.54mm_Vertical, symbol Connector_Generic:Conn_02x05_Odd_Even
- added J21: I2C connector, Connector_PinHeader_2.54mm:PinHeader_2x03_P2.54mm_Vertical, symbol Connector_Generic:Conn_02x03_Odd_Even
- added J22: NC, Connector:Tag-Connect_TC2050-IDC-FP_2x05_P1.27mm_Vertical, symbol Connector_Generic:Conn_02x05_Odd_Even
- added J28: 6x2 2.54mm header, Connector_PinHeader_2.54mm:PinHeader_2x06_P2.54mm_Vertical, symbol Connector_Generic:Conn_02x06_Odd_Even
- added R109, R110, R111, R112: 470, Resistor_SMD:R_0402_1005Metric, symbol Device:R
- added Y1: 25 Mhz Crystal +/- 10ppm, Oscillator:Oscillator_SMD_EuroQuartz_XO32-4Pin_3.2x2.5mm, symbol Device:Crystal_GND24
- C10: MPN (none) -> CL10A225KP8NNNC
- C14, C15, C16, C17, C18, C7: footprint Capacitor_SMD:C_0603_1608Metric -> Capacitor_SMD:C_0402_1005Metric; MPN (none) -> CL05B104K05NNNC; MPN2 (none) -> TCC0402X7R104M160AT
- D1: Link (none) -> https://eu.mouser.com/ProductDetail/onsemi-Fairchild/1N4148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; MPN (none) -> 1N4148WT
- D2, D3, D4, D5: MPN (none) -> LTST-C190KRKT
- R1, R2: footprint Resistor_SMD:R_0603_1608Metric -> Resistor_SMD:R_0402_1005Metric; MFN RT0603BRE0750RL -> RC0402JR-0750RL; MPN (none) -> RC0402JR-0750RL
- R10: value 4k7 -> 10k; footprint Resistor_SMD:R_0603_1608Metric -> Resistor_SMD:R_0402_1005Metric; MFN RTT034701FTP -> RTT02103JTH; MPN (none) -> RTT02103JTH
- R15, R22: footprint Resistor_SMD:R_0603_1608Metric -> Resistor_SMD:R_0402_1005Metric; MFN CRCW060310K0FKEA -> RTT02103JTH; MPN (none) -> RTT02103JTH
- R16, R20, R21, R23: value 1k -> 470; footprint Resistor_SMD:R_0603_1608Metric -> Resistor_SMD:R_0402_1005Metric; MFN RTT031001FTP -> RTT02471JTH; MPN (none) -> RTT02471JTH
- SW1: MPN (none) -> K2-1102BQ-C4CW-01
- SW2: footprint Button_Switch_SMD:SW_SPST_B3S-1000 -> Button_Switch_THT:SW_Tactile_SPST_Angled_PTS645Vx58-2LFS; MFN K2-1102SP-C4SC-04 -> K2-1102BQ-C4CW-01; MPN (none) -> K2-1102BQ-C4CW-01
- SW3: MPN (none) -> K2-1102SP-C4SC-04
- U1: MPN (none) -> STM32F411CEU6
Connections:
- net +3.3V: now also C73.2, C74.1, C75.2, C76.1, J20.1 (Pin_1), J21.1 (Pin_1), J21.5 (Pin_5), J22.1 (Pin_1), J28.2 (Pin_2), J28.4 (Pin_4), J28.6 (Pin_6), J28.8 (Pin_8)
- net BUTTON: now also J28.10 (Pin_10)
- net CURRENT_SENSE: now also TP6.1
- net GND: now also C66.1, C67.1, C73.1, C74.2, C75.1, C76.2, J20.4 (Pin_4), J20.9 (Pin_9), J21.3 (Pin_3), J22.10 (Pin_10), J22.2 (Pin_2), J22.4 (Pin_4), J22.6 (Pin_6), J22.7 (Pin_7), J22.8 (Pin_8), J28.11 (Pin_11), J28.9 (Pin_9), R109.1, Y1.2, Y1.4
- net GNDA: now also GNDA1.1
- net I2C1_SCL: now also J21.2 (Pin_2)
- net I2C1_SDA: now also J21.4 (Pin_4)
- net IRQ_IN: now also J20.6 (Pin_6), J21.6 (Pin_6)
- net LED0: now also R112.1
- net LED1: now also R111.1
- net LED2: now also R110.1
- net NRST: now also J22.9 (Pin_9), J28.12 (Pin_12), TP5.1
- net SPI2_MISO: now also J20.5 (Pin_5)
- net SPI2_MOSI: now also J20.3 (Pin_3)
- net SPI2_NSS: now also J20.10 (Pin_10)
- net SPI2_SCK: now also J20.7 (Pin_7)
- net SWCLK: now also J22.5 (Pin_5)
- net SWDIO: now also J22.3 (Pin_3)
- net USB_OEn: now also TP1.1
- net USB_SEL: now also TP2.1
- net XTALI: now also U1.5 (PH0), C66.2, Y1.1; no longer U1.6 (PH1)
- net XTALO: now also U1.6 (PH1), C67.2, Y1.3; no longer U1.5 (PH0)
- net nRESET_OUT: now also J20.2 (Pin_2)
- net FT2232_EECLK: now reaches U1.13 (PA3)
- net FT2232_EECS: now reaches U1.19 (PB1)
- net FT2232_EEDATA: now reaches U1.31 (PA10)
- net _DN renamed DN
- net _DP renamed DP
- new net: J28.7 (Pin_7), R112.2
- new net: J28.3 (Pin_3), R110.2
- new net: J28.1 (Pin_1), R109.2
- new net: J28.5 (Pin_5), R111.2
Other:
- added sheet FT2232 (ft2232_interface.kicad_sch)
- added sheet Power (power_supplies.kicad_sch)
- added sheet USB 3.2 Gen2 front-hub (usb3_hub.kicad_sch)
- sheet USB_STORAGE_MUX ports: added HUB_PRTCTL, SHOST_DN, SHOST_DP, SHOST_SSRXN, SHOST_SSRXP, SHOST_SSTXN, SHOST_SSTXP; removed none
- sheet board_control ports: added V_IN_ATX12, V_IN_ATX5; removed none
- note added: "LEDS"
- note added: "RESET"
- moved on the sheet: C10, C14, C15, C16, C17, C18, C7, D1, D2, D3, D4, GND1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
